File: hardware/food_dispenser.sch (EAGLE design)
At the start: 7 parts, among them IC1 ESP-12E/F, IC2 1182-A4988

Commit message: feat: add gnd plate, pin names and logo to board
Connections:
- net N$4 renamed GND
Changed lines of the file:
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@@
 </segment>
 </net>
-<net name="N$4" class="0">
+<net name="GND" class="0">
 <segment>
 <pinref part="JP3" gate="G$1" pin="2"/>
